File: AppleJoy.kicad_pcb (KiCad board)
At the start: 2 copper layers, 33 x 33 mm, 27 parts, among them J1 Atari, J2 Apple, Q1 BC558, Q2 BC558, Q3 BC558, Q4 BC558, Q5 BC558, Q6 BC558

Commit message: Slight tweaks for PCBway.
Other:
- board text added: "Apple II joystick adaptor"
- board text added: "Original design by Tor Arne Hustvedt 2021"
- board text added: "Revised layout by Chris RYU 2023"
- board text removed: "Apple IIe joystick adaptor"
- board text removed: "Tor Arne Hustvedt - 2021"
Changed lines of the file:
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@@
   (gr_arc (start 85.212 47.492) (mid 85.797786 46.077786) (end 87.212 45.492)
     (stroke (width 0.1) (type solid)) (layer "Edge.Cuts"))
-  (gr_text "Tor Arne Hustvedt - 2021" (at 86.017 62.478 -90) (layer "B.SilkS")
-    (effects (font (size 1 1) (thickness 0.15)) (justify mirror))
+  (gr_text "Original design by Tor Arne Hustvedt 2021" (at 86.128 63.33 90) (layer "B.SilkS")
+    (effects (font (size 0.75 0.75) (thickness 0.15)) (justify mirror))
   )
   (gr_text "Joystick/Gamepad" (at 108.338 73.79) (layer "B.SilkS")
     (effects (font (size 1 1) (thickness 0.15)) (justify left bottom mirror))
   )
+  (gr_text "Revised layout by Chris RYU 2023" (at 89.788 54.02 90) (layer "B.SilkS")
+    (effects (font (size 0.75 0.75) (thickness 0.1875) bold) (justify left bottom mirror))
+  )
   (gr_text "Apple" (at 103.908 50.92) (layer "B.SilkS")
     (effects (font (size 1 1) (thickness 0.15)) (justify left bottom mirror))
   )
-  (gr_text "Apple IIe joystick adaptor" (at 117.259 63.367 90) (layer "B.SilkS")
+  (gr_text "Apple II joystick adaptor" (at 117.259 63.367 90) (layer "B.SilkS")
     (effects (font (size 1 1) (thickness 0.15)) (justify mirror))
   )
